Commit message: right before gripper

File: pipebot_config/urdf/pipebot.urdf (robot description, URDF)
Before this commit: robot pipebot, 23 links, 22 joints
Links:
- added link d435_link, mass 0.01
- added link imu_link, mass 0.01; visual sphere radius=0.03
- added link l515_link, mass 0.01
- added link l515_link_back, mass 0.01; visual sphere radius=0.03
- added link t265_link, mass 0.01
- link ARM_1_1: geometry collision sphere radius=0.05; visual mesh filename=package://pipebot_config/meshes/ARM_1_1.stl scale=0.001 0.001 0.001
- link ARM_2_1: geometry collision cylinder length=0.26 radius=0.025; visual mesh filename=package://pipebot_config/meshes/ARM_2_1.stl scale=0.001 0.001 0.001
- link ARM_3_1: geometry collision cylinder length=0.16 radius=0.035; visual mesh filename=package://pipebot_config/meshes/ARM_3_1.stl scale=0.001 0.001 0.001
- link ARM_4_1: geometry visual mesh filename=package://pipebot_config/meshes/ARM_4_1.stl scale=0.001 0.001 0.001
- link ARM_5_1: geometry collision cylinder length=0.16 radius=0.03; visual mesh filename=package://pipebot_config/meshes/ARM_5_1.stl scale=0.001 0.001 0.001
- link ARM_6_1: geometry visual mesh filename=package://pipebot_config/meshes/ARM_6_1.stl scale=0.001 0.001 0.001
- link BL_calf_1: geometry collision cylinder length=0.26 radius=0.02; visual mesh filename=package://pipebot_config/meshes/BL_calf_1.stl scale=0.001 0.001 0.001
- link BL_foot_1: geometry collision sphere radius=0.03; visual mesh filename=package://pipebot_config/meshes/BL_foot_1.stl scale=0.001 0.001 0.001
- link BL_hip_2: geometry visual mesh filename=package://pipebot_config/meshes/BL_hip_2.stl scale=0.001 0.001 0.001
- link BL_thigh_1: geometry collision cylinder length=0.22 radius=0.035; visual mesh filename=package://pipebot_config/meshes/BL_thigh_1.stl scale=0.001 0.001 0.001
- link BR_calf_1: geometry collision cylinder length=0.26 radius=0.02; visual mesh filename=package://pipebot_config/meshes/BR_calf_1.stl scale=0.001 0.001 0.001
- link BR_foot_4: geometry collision sphere radius=0.03; visual mesh filename=package://pipebot_config/meshes/BR_foot_4.stl scale=0.001 0.001 0.001
- link BR_hip_1: geometry visual mesh filename=package://pipebot_config/meshes/BR_hip_1.stl scale=0.001 0.001 0.001
- link BR_thigh_1: geometry collision cylinder length=0.22 radius=0.035; visual mesh filename=package://pipebot_config/meshes/BR_thigh_1.stl scale=0.001 0.001 0.001
- link FL_calf_1: geometry collision cylinder length=0.26 radius=0.02; visual mesh filename=package://pipebot_config/meshes/FL_calf_1.stl scale=0.001 0.001 0.001
- link FL_foot_1: geometry collision sphere radius=0.03; visual mesh filename=package://pipebot_config/meshes/FL_foot_1.stl scale=0.001 0.001 0.001
- link FL_hip_1: geometry visual mesh filename=package://pipebot_config/meshes/FL_hip_1.stl scale=0.001 0.001 0.001
- link FL_thigh_1: geometry collision cylinder length=0.22 radius=0.035; visual mesh filename=package://pipebot_config/meshes/FL_thigh_1.stl scale=0.001 0.001 0.001
- link FR_calf_2: geometry collision cylinder length=0.26 radius=0.02; visual mesh filename=package://pipebot_config/meshes/FR_calf_2.stl scale=0.001 0.001 0.001
- link FR_foot_1: geometry collision sphere radius=0.03; visual mesh filename=package://pipebot_config/meshes/FR_foot_1.stl scale=0.001 0.001 0.001
- link FR_hip_1: geometry visual mesh filename=package://pipebot_config/meshes/FR_hip_1.stl scale=0.001 0.001 0.001
- link FR_thigh_2: geometry collision cylinder length=0.22 radius=0.035; visual mesh filename=package://pipebot_config/meshes/FR_thigh_2.stl scale=0.001 0.001 0.001
- link base_link: geometry collision box size=0.532 0.285 0.135; visual mesh filename=package://pipebot_config/meshes/base_link.stl scale=0.001 0.001 0.001
Joints:
- added joint cam_fixed_d435: type fixed, parent ARM_6_1, child d435_link, origin xyz=-0.04 0 0.05 rpy=0 -1.5708 0, axis 1 0 0
- added joint cam_fixed_l515: type fixed, parent base_link, child l515_link, origin xyz=0.28 0 0.08 rpy=0 0 0, axis 1 0 0
- added joint cam_fixed_l515_back: type fixed, parent base_link, child l515_link_back, origin xyz=-0.28 0 0.08 rpy=0 0 3.141592, axis 1 0 0
- added joint cam_fixed_t265: type fixed, parent base_link, child t265_link, origin xyz=0.285 0 0.1 rpy=0 0 0, axis 1 0 0
- added joint imu_base: type fixed, parent base_link, child imu_link, origin xyz=0 0 0 rpy=0 0 0
- joint BL_calf_joint: limit (none) -> lower=-3.0 upper=3.0 effort=80 velocity=15.0
- joint BL_hip_joint: limit (none) -> lower=-3.0 upper=3.0 effort=80 velocity=15.0
- joint BL_thigh_joint: limit (none) -> lower=-3.0 upper=3.0 effort=80 velocity=15.0
- joint BR_calf_joint: axis 0.0 -1.0 0.0 -> 0.0 1.0 0.0; limit (none) -> lower=-3.0 upper=3.0 effort=80 velocity=15.0
- joint BR_hip_joint: limit (none) -> lower=-3.0 upper=3.0 effort=80 velocity=15.0
- joint BR_thigh_joint: axis 0.0 -1.0 0.0 -> 0.0 1.0 0.0; limit (none) -> lower=-3.0 upper=3.0 effort=80 velocity=15.0
- joint FL_calf_joint: limit (none) -> lower=-3.0 upper=3.0 effort=80 velocity=15.0
- joint FL_hip_joint: axis -1.0 -0.0 0.0 -> 1.0 -0.0 0.0; limit (none) -> lower=-3.0 upper=3.0 effort=80 velocity=15.0
- joint FL_thigh_joint: limit (none) -> lower=-3.0 upper=3.0 effort=80 velocity=15.0
- joint FR_calf_joint: axis 0.0 -1.0 -0.0 -> 0.0 1.0 -0.0; limit (none) -> lower=-3.0 upper=3.0 effort=80 velocity=15.0
- joint FR_hip_joint: axis -1.0 -0.0 0.0 -> 1.0 -0.0 0.0; limit (none) -> lower=-3.0 upper=3.0 effort=80 velocity=15.0
- joint FR_thigh_joint: axis 0.0 -1.0 -0.0 -> 0.0 1.0 -0.0; limit (none) -> lower=-3.0 upper=3.0 effort=80 velocity=15.0
- joint arm_1_joint: limit (none) -> lower=-3.0 upper=3.0 effort=80 velocity=15.0
- joint arm_2_joint: limit (none) -> lower=-3.0 upper=3.0 effort=80 velocity=15.0
- joint arm_3_joint: limit (none) -> lower=-3.0 upper=3.0 effort=80 velocity=15.0
- joint arm_4_joint: limit (none) -> lower=-3.0 upper=3.0 effort=80 velocity=15.0
- joint arm_5_joint: limit (none) -> lower=-3.0 upper=3.0 effort=80 velocity=15.0
- joint arm_6_joint: limit (none) -> lower=-3.0 upper=3.0 effort=80 velocity=15.0

Commit message: finished

File: pipebot_config/urdf/pipebot.urdf (robot description, URDF)
Before this commit: robot pipebot, 28 links, 27 joints
Links:
- added link left_inner_finger, mass 0.0104003125914103; collision box size=0.015 0.015 0.05; visual mesh filename=package://pipebot_config/meshes/visual/robotiq_arg2f_140_in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
- added link left_inner_finger_pad; collision box size=0.03 0.07 0.0075; visual box size=0.027 0.065 0.0075
- added link left_inner_knuckle, mass 0.0271177346495152; collision box size=0.03 0.015 0.11; visual mesh filename=package://pipebot_config/meshes/visual/robotiq_arg2f_140_in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
- added link left_outer_finger, mass 0.022614240507152; collision box size=0.03 0.01 0.1; visual mesh filename=package://pipebot_config/meshes/visual/robotiq_arg2f_140_ou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
- added link left_outer_knuckle, mass 0.00853198276973456; visual mesh filename=package://pipebot_config/meshes/visual/robotiq_arg2f_140_ou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
- added link right_inner_finger, mass 0.0104003125914103; collision box size=0.015 0.015 0.05; visual mesh filename=package://pipebot_config/meshes/visual/robotiq_arg2f_140_in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
- added link right_inner_finger_pad; collision box size=0.03 0.07 0.0075; visual box size=0.027 0.065 0.0075
- added link right_inner_knuckle, mass 0.0271177346495152; collision box size=0.03 0.015 0.11; visual mesh filename=package://pipebot_config/meshes/visual/robotiq_arg2f_140_in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
- added link right_outer_finger, mass 0.022614240507152; collision box size=0.03 0.01 0.1; visual mesh filename=package://pipebot_config/meshes/visual/robotiq_arg2f_140_ou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
- added link right_outer_knuckle, mass 0.00853198276973456; visual mesh filename=package://pipebot_config/meshes/visual/robotiq_arg2f_140_ou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
- added link robotiq_arg2f_base_link, mass 0.22652; collision cylinder length=0.08 radius=0.04; visual mesh filename=package://pipebot_config/meshes/visual/robotiq_arg2f_base_l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
- link imu_link: geometry 
- link l515_link_back: geometry 
Joints:
- added joint arm_6_finger_joint: type fixed, parent ARM_6_1, child robotiq_arg2f_base_link, origin xyz=0.0 0.0 0.02 rpy=0 0 0
- added joint finger_joint: type revolute, parent robotiq_arg2f_base_link, child left_outer_knuckle, origin xyz=0 -0.030601 0.054905 rpy=2.29579632679 0 0, axis -1 0 0, limit lower=0 upper=0.7 effort=1000 velocity=2.0
- added joint left_inner_finger_joint: type revolute, parent left_outer_finger, child left_inner_finger, origin xyz=0 0.0817554015893473 -0.0282203446692936 rpy=-0.725 0 0, axis -1 0 0, limit lower=-0.8757 upper=0.0 effort=1000 velocity=2.0
- added joint left_inner_finger_pad_joint: type fixed, parent left_inner_finger, child left_inner_finger_pad, origin xyz=0 0.0457554015893473 -0.0272203446692936 rpy=0 0 0, axis 0 0 1
- added joint left_inner_knuckle_joint: type revolute, parent robotiq_arg2f_base_link, child left_inner_knuckle, origin xyz=0 -0.0127 0.06142 rpy=2.29579632679 0 0.0, axis -1 0 0, limit lower=0 upper=0.8757 effort=1000 velocity=2.0
- added joint left_outer_finger_joint: type fixed, parent left_outer_knuckle, child left_outer_finger, origin xyz=0 0.01821998610742 0.0260018192872234 rpy=0 0 0, axis 1 0 0
- added joint right_inner_finger_joint: type revolute, parent right_outer_finger, child right_inner_finger, origin xyz=0 0.0817554015893473 -0.0282203446692936 rpy=-0.725 0 0, axis -1 0 0, limit lower=-0.8757 upper=0.0 effort=1000 velocity=2.0
- added joint right_inner_finger_pad_joint: type fixed, parent right_inner_finger, child right_inner_finger_pad, origin xyz=0 0.0457554015893473 -0.0272203446692936 rpy=0 0 0, axis 0 0 1
- added joint right_inner_knuckle_joint: type revolute, parent robotiq_arg2f_base_link, child right_inner_knuckle, origin xyz=0 0.0127 0.06142 rpy=2.29579632679 0 -3.14159265359, axis -1 0 0, limit lower=0 upper=0.8757 effort=1000 velocity=2.0
- added joint right_outer_finger_joint: type fixed, parent right_outer_knuckle, child right_outer_finger, origin xyz=0 0.01821998610742 0.0260018192872234 rpy=0 0 0, axis 1 0 0
- added joint right_outer_knuckle_joint: type revolute, parent robotiq_arg2f_base_link, child right_outer_knuckle, origin xyz=0 0.030601 0.054905 rpy=2.29579632679 0 3.14159265359, axis -1 0 0, limit lower=0 upper=0.725 effort=1000 velocity=2.0

Commit message: logo and text changed

File: pipebot_config/urdf/pipebot.urdf (robot description, URDF)
Before this commit: robot pipebot, 39 links, 38 joints
Joints:
- joint BL_foot_fixed: limit (none) -> lower=0 upper=0 effort=1000 velocity=6.5; type fixed -> revolute
- joint BR_foot_fixed: limit (none) -> lower=0 upper=0 effort=1000 velocity=6.5; type fixed -> revolute
- joint FL_foot_fixed: limit (none) -> lower=0 upper=0 effort=1000 velocity=6.5; type fixed -> revolute
- joint FR_foot_fixed: limit (none) -> lower=0 upper=0 effort=1000 velocity=6.5; type fixed -> revolute
- joint arm_6_finger_joint: limit (none) -> lower=0 upper=0 effort=1000 velocity=6.5; type fixed -> revolute

Commit message: grasph plugin

File: pipebot_config/urdf/pipebot.urdf (robot description, URDF)
Before this commit: robot pipebot, 39 links, 38 joints
Joints:
- joint BL_foot_fixed: limit lower=0 upper=0 effort=1000 velocity=6.5 -> (none); type revolute -> fixed
- joint BR_foot_fixed: limit lower=0 upper=0 effort=1000 velocity=6.5 -> (none); type revolute -> fixed
- joint FL_foot_fixed: limit lower=0 upper=0 effort=1000 velocity=6.5 -> (none); type revolute -> fixed
- joint FR_foot_fixed: limit lower=0 upper=0 effort=1000 velocity=6.5 -> (none); type revolute -> fixed
- joint arm_6_finger_joint: limit lower=0 upper=0 effort=1000 velocity=6.5 -> (none); type revolute -> fixed
